File: senseboard.kicad_pcb (KiCad board)
At the start: 6 copper layers, 60 x 100 mm, 105 parts, among them J1 USB_C_Receptacle_USB2.0_16P, J2 Screw_Terminal_01x02, J3 DM3AT-SF-PEJM5, J4 Conn_01x04, J5 Conn_01x08, U1 USBLC6-2SC6, U10 EMIF06-MSD02N16, U11 BME690, U2 TPS62849DLCR, U3 TPS62849DLCR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

Commit message: final layout mods and added a couple more bulk caps
Parts:
- added C35: 4.7uF, Capacitor_SMD:C_0603_1608Metric, F.Cu at (129.1, 75.9)
- added C36: 10uF, Capacitor_SMD:C_0805_2012Metric, F.Cu at (116.5, 109.4)
- added C37: 4.7uF, Capacitor_SMD:C_0603_1608Metric, F.Cu at (119.8, 93.9)
- added C38: 4.7uF, Capacitor_SMD:C_0603_1608Metric, F.Cu at (87.6, 122.2)
- R1: value 0 -> 10k
- moved G*** 1.80 mm to (124.9, 137.0)
- moved J5 0.10 mm to (100.2, 168.5)
Routing:
- net +3V3_2: track 18.3 -> 21.7 mm, vias 31 -> 34
- net +3V3_1: track 52.7 -> 56.0 mm
- net GND: track 78.7 -> 81.2 mm
- net /I2C2_SDA: track 81.2 -> 81.8 mm

Commit message: added first turn of gerbers and drill files, added boms and placement files
Parts:
- D2, D4: footprint Diode_SMD:D_SMP_DO-220AA -> Diode_SMD:D_SMA
- moved D2 1.22 mm to (107.6, 160.2)
- moved D4 1.22 mm to (99.6, 160.2)
- moved C3 0.20 mm to (123.2, 158.8)
- moved C4 0.20 mm to (118.4, 154.2)
- moved J1 0.20 mm to (125.5, 166.0)
- moved R2 0.20 mm to (131.5, 165.6)
- moved R3 0.20 mm to (131.5, 163.6)
- moved U1 0.20 mm to (125.5, 158.9)
- moved C15 0.20 mm to (96.1, 158.2)
- moved R22 0.20 mm to (97.2, 160.2)
- moved R23 0.20 mm to (97.2, 158.2)
- moved C5 0.20 mm to (122.0, 154.9)
- moved F1 0.20 mm to (119.9, 154.9)
- moved FB1 0.20 mm to (124.6, 154.0)
- moved R4 0.20 mm to (124.5, 155.8)
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