File: senseboard.kicad_pcb (KiCad board)
At the start: 6 copper layers, 60 x 100 mm, 109 parts, among them J1 USB_C_Receptacle_USB2.0_16P, J2 Screw_Terminal_01x02, J3 DM3AT-SF-PEJM5, J4 Conn_01x04, J5 Conn_01x08, U1 USBLC6-2SC6, U10 EMIF06-MSD02N16, U11 BME690, U2 TPS62849DLCR, U3 TPS62849DLCR, U4 SCD41-D-R2, U5 SGP41-D-R4, U6 SGP41-D-R4, U7 SHT4x, U8 STM32L4Q5CGUx, U9 RFM95W-915S2, Y1 Crystal_GND3, Y2 Crystal

Commit message: added updated step with components and traces
Connections:
- net /SD_CLK renamed /Interfaces/SD_CLK
- net /SD_CMD renamed /Interfaces/SD_CMD
- net /SD_D0 renamed /Interfaces/SD_D0
- net /SD_D1 renamed /Interfaces/SD_D1
- net /SD_D2 renamed /Interfaces/SD_D2
- net /SD_D3 renamed /Interfaces/SD_D3
