File: senseboard.kicad_sch (KiCad schematic)
At the start: 105 parts, among them J1 USB_C_Receptacle_USB2.0_16P, J2 Screw_Terminal_01x02, J3 DM3AT-SF-PEJM5, J4 Conn_01x04, J5 Conn_01x08, U1 USBLC6-2SC6, U10 EMIF06-MSD02N16, U11 BME690, U2 TPS62849DLCR, U3 TPS62849DLCR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

Commit message: added first turn of gerbers and drill files, added boms and placement files
Parts:
- D2, D4: footprint Diode_SMD:D_SMP_DO-220AA -> Diode_SMD:D_SMA
Changed lines of the file:
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@@
 			)
 		)
-		(property "Footprint" "Diode_SMD:D_SMP_DO-220AA"
+		(property "Footprint" "Diode_SMD:D_SMA"
 			(at 53.34 133.35 0)
 			(hide yes)
@@
 						(field
 							(name "Value")
-							(value "STPS1L30MF")
+							(value "STPS1L30A")
 						)
 					)
@@
 			)
 		)
-		(property "Footprint" "Diode_SMD:D_SMP_DO-220AA"
+		(property "Footprint" "Diode_SMD:D_SMA"
 			(at 50.8 71.12 0)
 			(hide yes)
@@
 						(field
 							(name "Value")
-							(value "STPS1L30MF")
+							(value "STPS1L30A")
 						)
 					)
