File: senseboard.kicad_sch (KiCad schematic)
At the start: 105 parts, among them J1 USB_C_Receptacle_USB2.0_16P, J2 Screw_Terminal_01x02, J3 DM3AT-SF-PEJM5, J4 Conn_01x04, J5 Conn_01x08, U1 USBLC6-2SC6, U10 EMIF06-MSD02N16, U11 BME690, U2 TPS62849DLCR, U3 TPS62849DLCR, U4 SCD41-D-R2, U5 SGP41-D-R4, U6 SGP41-D-R4, U7 SHT4x, U8 STM32L4Q5CGUx, U9 RFM95W-915S2, Y1 Crystal_GND3, Y2 Crystal

Commit message: cleaned schematic for interview
Parts:
- removed C14, C21, C4: 0.1uF, Capacitor_SMD:C_0402_1005Metric, symbol Device:C
- removed C3: 10nF, Capacitor_SMD:C_0402_1005Metric, symbol Device:C
- removed C34: 10uF, Capacitor_SMD:C_0805_2012Metric, symbol Device:C
- removed C5: 4.7uF, Capacitor_SMD:C_0805_2012Metric, symbol Device:C
- removed F1: Polyfuse, Fuse:Fuse_0805_2012Metric, symbol Device:Polyfuse
- removed FB1: FerriteBead, Inductor_SMD:L_0603_1608Metric, symbol Device:FerriteBead
- removed J1: USB_C_Receptacle_USB2.0_16P, Connector_USB:USB_C_Receptacle_G-Switch_GT-USB-7010ASV, symbol Connector:USB_C_Receptacle_USB2.0_16P
- removed J3: DM3AT-SF-PEJM5, DM3AT_SF_PEJM5:HRS_DM3AT-SF-PEJM5, symbol DM3AT-SF-PEJM5:DM3AT-SF-PEJM5
- removed J4: Conn_01x04, Connector_PinHeader_2.54mm:PinHeader_1x04_P2.54mm_Vertical, symbol Connector_Generic:Conn_01x04
- removed J5: Conn_01x08, Connector_PinHeader_2.54mm:PinHeader_1x08_P2.54mm_Vertical, symbol Connector_Generic:Conn_01x08
- removed R2, R3: 5.1k, Resistor_SMD:R_0402_1005Metric, symbol Device:R
- removed R4, R5: 0, Resistor_SMD:R_0402_1005Metric, symbol Device:R
- removed U1: USBLC6-2SC6, Package_TO_SOT_SMD:SOT-23-6, symbol Power_Protection:USBLC6-2SC6
- removed U10: EMIF06-MSD02N16, EMIF06_MSD02N16:MICROQFN16_1P25X3P55X0P4_STM, symbol EMIF06_MSD02N16:EMIF06-MSD02N16
Connections:
- no-connect marks 3 -> 0
Other:
- added sheet Interfaces (interfaces.kicad_sch)
- moved on the sheet: AE1, BT1, C1, C10, C11, C12, C13, C15, C16, C17, C18, C19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
